File: hardware/board/mkey.kicad_sch (KiCad schematic)
At the start: 163 parts, among them J1 USB_C_REP_2.0, J2 24 pin LCD FPC connector, SW1 SW_Push, SW2 SW_Push, U1 ESP32-S3-WROOM-1, U5 SY8088

Commit message: fix that the USB pins were swapped
Connections:
- net USB_D+: now also D69.2 (K), J1.A6 (D+), J1.B6 (D+); no longer D69.3 (K), J1.A7 (D-), J1.B7 (D-)
- net USB_D-: now also D69.3 (K), J1.A7 (D-), J1.B7 (D-); no longer D69.2 (K), J1.A6 (D+), J1.B6 (D+)
Changed lines of the file:
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@@
     )
   )
-  (global_label "USB_D+" (shape bidirectional) (at 119.38 233.68 0) (fields_autoplaced)
+  (global_label "USB_D+" (shape bidirectional) (at 119.38 238.76 0) (fields_autoplaced)
     (effects (font (size 1.27 1.27)) (justify left))
-    (property "Intersheetrefs" "${INTERSHEET_REFS}" (at 130.2041 233.68 0)
+    (property "Intersheetrefs" "${INTERSHEET_REFS}" (at 130.2041 238.76 0)
       (effects (font (size 1.27 1.27)) (justify left) hide)
     )
@@
     )
   )
-  (global_label "USB_D-" (shape bidirectional) (at 119.38 238.76 0) (fields_autoplaced)
+  (global_label "USB_D-" (shape bidirectional) (at 119.38 233.68 0) (fields_autoplaced)
     (effects (font (size 1.27 1.27)) (justify left))
-    (property "Intersheetrefs" "${INTERSHEET_REFS}" (at 130.2041 238.76 0)
+    (property "Intersheetrefs" "${INTERSHEET_REFS}" (at 130.2041 233.68 0)
       (effects (font (size 1.27 1.27)) (justify left) hide)
     )
