File: hardware/board/mkey.kicad_pcb (KiCad board)
At the start: 2 copper layers, 346.2 x 95.5 mm, 171 parts, among them J1 USB_C_REP_2.0, J2 24 pin LCD FPC connector, SW0 SW_Push, SW1 SW_Push, U1 ESP32-S3-WROOM-1, U2 SY8088

Commit message: hw: fix sio labels
Connections:
- net LCD_SIO4 renamed LCD_SIO2
Changed lines of the file:
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@@
   (net 109 "TP_INT")
   (net 110 "TP_SDA")
-  (net 111 "LCD_SIO4")
+  (net 111 "LCD_SIO2")
   (net 112 "LCD_D{slash}C")
   (net 113 "LCD_SIO3")
@@
     (fp_arc (start -46.63125 7.500001) (mid -46.777697 7.853554) (end -47.13125 8.000001)
       (stroke (width 0.05) (type solid)) (layer "Eco2.User"))
-    (fp_arc (start 46.63125 -5.499999) (mid 46.777693 -5.853571) (end 47.13125 -5.999999)
+    (fp_arc (start 46.63125 -5.499999) (mid 46.777699 -5.853535) (end 47.13125 -5.999999)
       (stroke (width 0.05) (type solid)) (layer "Eco2.User"))
-    (fp_arc (start 47.13125 8.000001) (mid 46.777729 7.853537) (end 46.63125 7.500001)
+    (fp_arc (start 47.13125 8.000001) (mid 46.777693 7.853543) (end 46.63125 7.500001)
       (stroke (width 0.05) (type solid)) (layer "Eco2.User"))
-    (fp_arc (start 52.880039 -5.999999) (mid 53.233567 -5.853539) (end 53.380039 -5.499999)
+    (fp_arc (start 52.880039 -5.999999) (mid 53.233602 -5.853545) (end 53.380039 -5.499999)
       (stroke (width 0.05) (type solid)) (layer "Eco2.User"))
-    (fp_arc (start 53.38125 7.500001) (mid 53.234806 7.853571) (end 52.88125 8.000001)
+    (fp_arc (start 53.38125 7.500001) (mid 53.2348 7.853536) (end 52.88125 8.000001)
       (stroke (width 0.05) (type solid)) (layer "Eco2.User"))
     (pad "" thru_hole circle (at -50.00625 -6.985 180) (size 4 4) (drill 3.048) (layers "*.Cu" "B.Mask"))
@@
     (fp_arc (start 8.53125 -5.499999) (mid 8.677685 -5.853565) (end 9.03125 -5.999999)
       (stroke (width 0.05) (type solid)) (layer "Eco2.User"))
-    (fp_arc (start 9.03125 8.000001) (mid 8.677729 7.853537) (end 8.53125 7.500001)
+    (fp_arc (start 9.03125 8.000001) (mid 8.677693 7.853543) (end 8.53125 7.500001)
       (stroke (width 0.05) (type solid)) (layer "Eco2.User"))
-    (fp_arc (start 14.780039 -5.999999) (mid 15.133567 -5.853539) (end 15.280039 -5.499999)
+    (fp_arc (start 14.780039 -5.999999) (mid 15.133602 -5.853545) (end 15.280039 -5.499999)
       (stroke (width 0.05) (type solid)) (layer "Eco2.User"))
-    (fp_arc (start 15.28125 7.500001) (mid 15.134806 7.853571) (end 14.78125 8.000001)
+    (fp_arc (start 15.28125 7.500001) (mid 15.1348 7.853536) (end 14.78125 8.000001)
       (stroke (width 0.05) (type solid)) (layer "Eco2.User"))
     (pad "" thru_hole circle (at -11.90625 -6.985) (size 4 4) (drill 3.048) (layers "*.Cu" "B.Mask"))
@@
       (net 113 "LCD_SIO3") (pinfunction "Pin_22") (pintype "passive") (thermal_bridge_angle 45))
     (pad "23" smd rect (at -1.17202 1.886 270) (size 0.2 0.4) (layers "F.Cu" "F.Paste" "F.Mask")
-      (net 111 "LCD_SIO4") (pinfunction "Pin_23") (pintype "passive") (thermal_bridge_angle 45))
+      (net 111 "LCD_SIO2") (pinfunction "Pin_23") (pintype "passive") (thermal_bridge_angle 45))
     (pad "24" smd rect (at -1.17202 2.286 270) (size 0.2 0.4) (layers "F.Cu" "F.Paste" "F.Mask")
       (net 112 "LCD_D{slash}C") (pinfunction "Pin_24") (pintype "passive") (thermal_bridge_angle 45))
@@
     (fp_arc (start 8.53125 -5.499999) (mid 8.677685 -5.853565) (end 9.03125 -5.999999)
       (stroke (width 0.05) (type solid)) (layer "Eco2.User"))
-    (fp_arc (start 9.03125 8.000001) (mid 8.677729 7.853537) (end 8.53125 7.500001)
+    (fp_arc (start 9.03125 8.000001) (mid 8.677693 7.853543) (end 8.53125 7.500001)
       (stroke (width 0.05) (type solid)) (layer "Eco2.User"))
-    (fp_arc (start 14.780039 -5.999999) (mid 15.133567 -5.853539) (end 15.280039 -5.499999)
+    (fp_arc (start 14.780039 -5.999999) (mid 15.133602 -5.853545) (end 15.280039 -5.499999)
       (stroke (width 0.05) (type solid)) (layer "Eco2.User"))
-    (fp_arc (start 15.28125 7.500001) (mid 15.134806 7.853571) (end 14.78125 8.000001)
+    (fp_arc (start 15.28125 7.500001) (mid 15.1348 7.853536) (end 14.78125 8.000001)
       (stroke (width 0.05) (type solid)) (layer "Eco2.User"))
     (pad "" thru_hole circle (at -11.90625 -6.985) (size 4 4) (drill 3.048) (layers "*.Cu" "B.Mask"))
@@
       (net 113 "LCD_SIO3") (pinfunction "GPIO7/TOUCH7/ADC1_CH6") (pintype "bidirectional"))
     (pad "8" smd rect (at -8.75 -0.63 180) (size 1.5 0.9) (layers "B.Cu" "B.Paste" "B.Mask")
-      (net 111 "LCD_SIO4") (pinfunction "GPIO15/U0RTS/ADC2_CH4/XTAL_32K_P") (pintype "bidirectional"))
+      (net 111 "LCD_SIO2") (pinfunction "GPIO15/U0RTS/ADC2_CH4/XTAL_32K_P") (pintype "bidirectional"))
     (pad "9" smd rect (at -8.75 -1.9 180) (size 1.5 0.9) (layers "B.Cu" "B.Paste" "B.Mask")
       (net 112 "LCD_D{slash}C") (pinfunction "GPIO16/U0CTS/ADC2_CH5/XTAL_32K_N") (pintype "bidirectional"))
