File: hardware/plate/plate.kicad_pcb (KiCad board)
At the start: 2 copper layers, 352.6 x 100.2 mm, 0 parts

Commit message: new plate with tabs, final order
Other:
- board size 352.6 x 100.2 mm -> 356.2 x 103.8 mm
